File: DB37breakout.kicad_sch (KiCad schematic)
At the start: 34 parts, among them J10 Conn_Coaxial, J11 Conn_Coaxial, J12 Conn_Coaxial, J13 Conn_Coaxial, J14 Conn_Coaxial, J15 Conn_Coaxial, J16 Conn_Coaxial, J17 Conn_Coaxial, J18 Conn_Coaxial, J19 Conn_Coaxial, J2 Conn_Coaxial, J20 Conn_Coaxial, J21 Conn_Coaxial, J22 Conn_Coaxial, J23 Conn_Coaxial, J24 Conn_Coaxial, J25 Conn_Coaxial, J26 Conn_Coaxial, J27 Conn_Coaxial, J28 Conn_Coaxial, J29 Conn_Coaxial, J3 Conn_Coaxial, J30 Conn_Coaxial, J31 Conn_Coaxial, J32 Conn_Coaxial, J33 Conn_Coaxial, J4 Conn_Coaxial, J5 Conn_Coaxial, J6 Conn_Coaxial, J7 Conn_Coaxial, J8 Conn_Coaxial, J9 Conn_Coaxial

Commit message: Changed BNC footprint to vertical Through Hole; redesigned board with greater space between traces and footprints; shortened board length and expanded board width to lightly less than a 2U space
Parts:
- added H1, H2, H3, H4, H5, H6: MountingHole, MountingHole:MountingHole_3mm, symbol Mechanical:MountingHole
- J10, J11, J12, J13, J14, J15, J16, J17, J18, J19, J2, J20, J21, J22, J23, J24, J25, J26, J27, J28, J29, J3, J30, J31, J32, J33, J4, J5, J6, J7, J8, J9: footprint Connector_Coaxial:BNC_Amphenol_031-5539_Vertical -> Connector_Coaxial:BNC_TEConnectivity_1478204_Vertical
